File: pico-swm-px26a-pcb.kicad_sch (KiCad schematic)
At the start: 12 parts, among them J1 Conn_01x03, J2 STLZ950/3G-5.08-V-GRÜN, U1 Pico, U2 4N35

Commit message: Add EEPROM
Parts:
- added U3: 25LCxxx, Package_DIP:DIP-8_W7.62mm, symbol Memory_EEPROM:25LCxxx
Connections:
- net +3V3: now also U3.8 (VCC)
- net GNDD: now also U3.4 (GND)
- net at U1.10 (GPIO7): now also U3.1 (~{CS})
- net at U1.11 (GPIO8): now also U3.2 (MISO)
- net at U1.12 (GPIO9): now also U3.7 (~{HOLD})
- net at U1.14 (GPIO10): now also U3.6 (SCK)
- net at U1.15 (GPIO11): now also U3.5 (MOSI)
- net at U1.16 (GPIO12): now also U3.3 (~{WP})
Changed lines of the file:
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@@
   )
   (no_connect (at 152.4 113.03))
+  (wire (pts (xy 74.93 82.55) (xy 74.93 95.25))
+    (stroke (width 0) (type default))
+  )
   (wire (pts (xy 128.27 72.39) (xy 130.81 72.39))
     (stroke (width 0) (type default))
   )
+  (wire (pts (xy 77.47 90.17) (xy 92.71 90.17))
+    (stroke (width 0) (type default))
+  )
   (wire (pts (xy 184.15 77.47) (xy 189.23 77.47))
     (stroke (width 0) (type default))
@@
     (stroke (width 0) (type default))
   )
+  (wire (pts (xy 77.47 92.71) (xy 92.71 92.71))
+    (stroke (width 0) (type default))
+  )
   (wire (pts (xy 186.69 110.49) (xy 186.69 120.65))
     (stroke (width 0) (type default))
@@
     (stroke (width 0) (type default))
   )
+  (wire (pts (xy 69.85 100.33) (xy 92.71 100.33))
+    (stroke (width 0) (type default))
+  )
   (wire (pts (xy 194.31 113.03) (xy 194.31 100.33))
     (stroke (width 0) (type default))
   )
+  (wire (pts (xy 81.28 105.41) (xy 92.71 105.41))
+    (stroke (width 0) (type default))
+  )
   (wire (pts (xy 189.23 110.49) (xy 189.23 113.03))
     (stroke (width 0) (type default))
   )
+  (wire (pts (xy 46.99 121.92) (xy 81.28 121.92))
+    (stroke (width 0) (type default))
+  )
+  (wire (pts (xy 69.85 102.87) (xy 92.71 102.87))
+    (stroke (width 0) (type default))
+  )
   (wire (pts (xy 148.59 118.11) (xy 148.59 120.65))
     (stroke (width 0) (type default))
@@
     (stroke (width 0) (type default))
   )
+  (wire (pts (xy 69.85 105.41) (xy 77.47 105.41))
+    (stroke (width 0) (type default))
+  )
   (wire (pts (xy 130.81 72.39) (xy 130.81 97.79))
     (stroke (width 0) (type default))
@@
     (stroke (width 0) (type default))
   )
+  (wire (pts (xy 41.91 105.41) (xy 41.91 80.01))
+    (stroke (width 0) (type default))
+  )
   (wire (pts (xy 90.17 97.79) (xy 90.17 110.49))
     (stroke (width 0) (type default))
@@
     (stroke (width 0) (type default))
   )
+  (wire (pts (xy 59.69 113.03) (xy 59.69 110.49))
+    (stroke (width 0) (type default))
+  )
+  (wire (pts (xy 77.47 80.01) (xy 77.47 90.17))
+    (stroke (width 0) (type default))
+  )
   (wire (pts (xy 153.67 77.47) (xy 153.67 80.01))
     (stroke (width 0) (type default))
@@
     (stroke (width 0) (type default))
   )
+  (wire (pts (xy 41.91 80.01) (xy 77.47 80.01))
+    (stroke (width 0) (type default))
+  )
+  (wire (pts (xy 59.69 92.71) (xy 59.69 95.25))
+    (stroke (width 0) (type default))
+  )
   (wire (pts (xy 107.95 120.65) (xy 107.95 124.46))
     (stroke (width 0) (type default))
@@
     (stroke (width 0) (type default))
   )
+  (wire (pts (xy 46.99 100.33) (xy 46.99 121.92))
+    (stroke (width 0) (type default))
+  )
+  (wire (pts (xy 81.28 121.92) (xy 81.28 105.41))
+    (stroke (width 0) (type default))
+  )
   (wire (pts (xy 148.59 100.33) (xy 148.59 102.87))
     (stroke (width 0) (type default))
@@
     (stroke (width 0) (type default))
   )
+  (wire (pts (xy 49.53 105.41) (xy 41.91 105.41))
+    (stroke (width 0) (type default))
+  )
   (wire (pts (xy 170.18 118.11) (xy 170.18 120.65))
     (stroke (width 0) (type default))
@@
     (stroke (width 0) (type default))
   )
+  (wire (pts (xy 77.47 105.41) (xy 77.47 92.71))
+    (stroke (width 0) (type default))
+  )
+  (wire (pts (xy 44.45 82.55) (xy 74.93 82.55))
+    (stroke (width 0) (type default))
+  )
   (wire (pts (xy 194.31 76.2) (xy 194.31 77.47))
     (stroke (width 0) (type default))
@@
     (stroke (width 0) (type default))
   )
+  (wire (pts (xy 49.53 102.87) (xy 44.45 102.87))
+    (stroke (width 0) (type default))
+  )
   (wire (pts (xy 90.17 72.39) (xy 90.17 85.09))
     (stroke (width 0) (type default))
@@
     (stroke (width 0) (type default))
   )
+  (wire (pts (xy 44.45 102.87) (xy 44.45 82.55))
+    (stroke (width 0) (type default))
+  )
+  (wire (pts (xy 74.93 95.25) (xy 92.71 95.25))
+    (stroke (width 0) (type default))
+  )
   (wire (pts (xy 128.27 67.31) (xy 134.62 67.31))
+    (stroke (width 0) (type default))
+  )
+  (wire (pts (xy 49.53 100.33) (xy 46.99 100.33))
     (stroke (width 0) (type default))
   )
@@
         (path "/9434df5a-8c9d-47a4-9450-184b012d901d"
           (reference "#PWR012") (unit 1)
+        )
+      )
+    )
+  )
+  (symbol (lib_id "power:GNDD") (at 59.69 113.03 0) (unit 1)
+    (in_bom yes) (on_board yes) (dnp no) (fields_autoplaced)
+    (property "Reference" "#PWR03" (at 59.69 119.38 0)
+      (effects (font (size 1.27 1.27)) hide)
+    )
+    (property "Value" "GNDD" (at 59.69 118.11 0)
+      (effects (font (size 1.27 1.27)))
+    )
+    (property "Footprint" "" (at 59.69 113.03 0)
+      (effects (font (size 1.27 1.27)) hide)
+    )
+    (property "Datasheet" "" (at 59.69 113.03 0)
+      (effects (font (size 1.27 1.27)) hide)
+    )
+    (pin "1")
+    (instances
+      (project "pico-swm-px26a-pcb"
+        (path "/9434df5a-8c9d-47a4-9450-184b012d901d"
+          (reference "#PWR03") (unit 1)
         )
       )
@@
         (path "/9434df5a-8c9d-47a4-9450-184b012d901d"
           (reference "#PWR011") (unit 1)
+        )
+      )
+    )
+  )
+  (symbol (lib_id "power:+3V3") (at 59.69 92.71 0) (unit 1)
+    (in_bom yes) (on_board yes) (dnp no) (fields_autoplaced)
+    (property "Reference" "#PWR01" (at 59.69 96.52 0)
+      (effects (font (size 1.27 1.27)) hide)
+    )
+    (property "Value" "+3V3" (at 59.69 88.9 0)
+      (effects (font (size 1.27 1.27)))
+    )
+    (property "Footprint" "" (at 59.69 92.71 0)
+      (effects (font (size 1.27 1.27)) hide)
+    )
+    (property "Datasheet" "" (at 59.69 92.71 0)
+      (effects (font (size 1.27 1.27)) hide)
+    )
+    (pin "1")
+    (instances
+      (project "pico-swm-px26a-pcb"
+        (path "/9434df5a-8c9d-47a4-9450-184b012d901d"
+          (reference "#PWR01") (unit 1)
         )
       )
@@
         )
       )
+    )
+  )
+  (symbol (lib_id "Memory_EEPROM:25LCxxx") (at 59.69 102.87 0) (unit 1)
+    (in_bom yes) (on_board yes) (dnp no) (fields_autoplaced)
+    (property "Reference" "U3" (at 61.8841 92.71 0)
+      (effects (font (size 1.27 1.27)) (justify left))
+    )
+    (property "Value" "25LCxxx" (at 61.8841 95.25 0)
+      (effects (font (size 1.27 1.27)) (justify left))
+    )
+    (property "Footprint" "Package_DIP:DIP-8_W7.62mm" (at 59.69 102.87 0)
+      (effects (font (size 1.27 1.27)) hide)
+    )
+    (property "Datasheet" "http://ww1.microchip.com/downloads/en/DeviceDoc/21832H.pdf" (at 59.69 102.87 0)
+      (effects (font (size 1.27 1.27)) hide)
+    )
+    (pin "1")
+    (pin "3")
+    (pin "2")
+    (pin "7")
+    (pin "5")
+    (pin "4")
+    (pin "6")
+    (pin "8")
+    (instances
+      (project "pico-swm-px26a-pcb"
+        (path "/9434df5a-8c9d-47a4-9450-184b012d901d"
+          (reference "U3") (unit 1)
+        )
+      )

Commit message: Add EEPROM cap
Parts:
- added C3: 33u, Capacitor_THT:CP_Radial_D5.0mm_P2.00mm, symbol Device:C_Polarized
Connections:
- net +3V3: now also C3.1
- net GNDD: now also C3.2
Changed lines of the file:
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@@
+    (stroke (width 0) (type default))
+  )
+  (wire (pts (xy 29.21 109.22) (xy 29.21 106.68))
     (stroke (width 0) (type default))
   )
@@
   )
   (wire (pts (xy 170.18 118.11) (xy 170.18 120.65))
+    (stroke (width 0) (type default))
+  )
+  (wire (pts (xy 29.21 96.52) (xy 29.21 99.06))
     (stroke (width 0) (type default))
   )
@@
     )
   )
+  (symbol (lib_id "power:+3V3") (at 29.21 96.52 0) (unit 1)
+    (in_bom yes) (on_board yes) (dnp no) (fields_autoplaced)
+    (property "Reference" "#PWR018" (at 29.21 100.33 0)
+      (effects (font (size 1.27 1.27)) hide)
+    )
+    (property "Value" "+3V3" (at 29.21 92.71 0)
+      (effects (font (size 1.27 1.27)))
+    )
+    (property "Footprint" "" (at 29.21 96.52 0)
+      (effects (font (size 1.27 1.27)) hide)
+    )
+    (property "Datasheet" "" (at 29.21 96.52 0)
+      (effects (font (size 1.27 1.27)) hide)
+    )
+    (pin "1")
+    (instances
+      (project "pico-swm-px26a-pcb"
+        (path "/9434df5a-8c9d-47a4-9450-184b012d901d"
+          (reference "#PWR018") (unit 1)
+        )
+      )
+    )
+  )
   (symbol (lib_id "Device:R") (at 148.59 106.68 0) (unit 1)
     (in_bom yes) (on_board yes) (dnp no) (fields_autoplaced)
@@
     )
   )
+  (symbol (lib_id "Device:C_Polarized") (at 29.21 102.87 0) (mirror y) (unit 1)
+    (in_bom yes) (on_board yes) (dnp no)
+    (property "Reference" "C3" (at 25.4 101.346 0)
+      (effects (font (size 1.27 1.27)) (justify left))
+    )
+    (property "Value" "33u" (at 25.4 103.886 0)
+      (effects (font (size 1.27 1.27)) (justify left))
+    )
+    (property "Footprint" "Capacitor_THT:CP_Radial_D5.0mm_P2.00mm" (at 28.2448 106.68 0)
+      (effects (font (size 1.27 1.27)) hide)
+    )
+    (property "Datasheet" "~" (at 29.21 102.87 0)
+      (effects (font (size 1.27 1.27)) hide)
+    )
+    (pin "1")
+    (pin "2")
+    (instances
+      (project "pico-swm-px26a-pcb"
+        (path "/9434df5a-8c9d-47a4-9450-184b012d901d"
+          (reference "C3") (unit 1)
+        )
+      )
+    )
+  )
   (symbol (lib_id "Mechanical:MountingHole") (at 39.37 171.45 0) (unit 1)
     (in_bom no) (on_board yes) (dnp no) (fields_autoplaced)
@@
         )
       )
+    )
+  )
+  (symbol (lib_id "power:GNDD") (at 29.21 109.22 0) (unit 1)
+    (in_bom yes) (on_board yes) (dnp no) (fields_autoplaced)
+    (property "Reference" "#PWR017" (at 29.21 115.57 0)
+      (effects (font (size 1.27 1.27)) hide)
+    )
+    (property "Value" "GNDD" (at 29.21 114.3 0)
+      (effects (font (size 1.27 1.27)))
+    )
+    (property "Footprint" "" (at 29.21 109.22 0)
+      (effects (font (size 1.27 1.27)) hide)
+    )
+    (property "Datasheet" "" (at 29.21 109.22 0)
+      (effects (font (size 1.27 1.27)) hide)
+    )
+    (pin "1")
+    (instances
+      (project "pico-swm-px26a-pcb"
+        (path "/9434df5a-8c9d-47a4-9450-184b012d901d"
+          (reference "#PWR017") (unit 1)
+        )
+      )

Commit message: Initial routing
Connections:
- net at U1.10 (GPIO7): no longer U3.1 (~{CS})
- net at U1.17 (GPIO13): now also U3.1 (~{CS})
Changed lines of the file:
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@@
-    (stroke (width 0) (type default))
-  )
-  (wire (pts (xy 77.47 90.17) (xy 92.71 90.17))
     (stroke (width 0) (type default))
   )
@@
     (stroke (width 0) (type default))
   )
+  (wire (pts (xy 49.53 100.33) (xy 46.99 100.33))
+    (stroke (width 0) (type default))
+  )
+  (wire (pts (xy 80.01 120.65) (xy 80.01 105.41))
+    (stroke (width 0) (type default))
+  )
   (wire (pts (xy 119.38 128.27) (xy 119.38 123.19))
     (stroke (width 0) (type default))
@@
     (stroke (width 0) (type default))
   )
+  (wire (pts (xy 49.53 105.41) (xy 44.45 105.41))
+    (stroke (width 0) (type default))
+  )
   (wire (pts (xy 130.81 110.49) (xy 130.81 120.65))
     (stroke (width 0) (type default))
@@
     (stroke (width 0) (type default))
   )
-  (wire (pts (xy 81.28 105.41) (xy 92.71 105.41))
-    (stroke (width 0) (type default))
-  )
   (wire (pts (xy 189.23 110.49) (xy 189.23 113.03))
     (stroke (width 0) (type default))
   )
-  (wire (pts (xy 46.99 121.92) (xy 81.28 121.92))
+  (wire (pts (xy 44.45 123.19) (xy 82.55 123.19))
+    (stroke (width 0) (type default))
+  )
+  (wire (pts (xy 44.45 102.87) (xy 49.53 102.87))
     (stroke (width 0) (type default))
   )
@@
     (stroke (width 0) (type default))
   )
+  (wire (pts (xy 46.99 100.33) (xy 46.99 120.65))
+    (stroke (width 0) (type default))
+  )
   (wire (pts (xy 189.23 113.03) (xy 194.31 113.03))
     (stroke (width 0) (type default))
@@
     (stroke (width 0) (type default))
   )
-  (wire (pts (xy 41.91 105.41) (xy 41.91 80.01))
-    (stroke (width 0) (type default))
-  )
   (wire (pts (xy 90.17 97.79) (xy 90.17 110.49))
     (stroke (width 0) (type default))
@@
     (stroke (width 0) (type default))
   )
-  (wire (pts (xy 77.47 80.01) (xy 77.47 90.17))
-    (stroke (width 0) (type default))
-  )
   (wire (pts (xy 153.67 77.47) (xy 153.67 80.01))
     (stroke (width 0) (type default))
@@
     (stroke (width 0) (type default))
   )
-  (wire (pts (xy 41.91 80.01) (xy 77.47 80.01))
-    (stroke (width 0) (type default))
-  )
   (wire (pts (xy 59.69 92.71) (xy 59.69 95.25))
     (stroke (width 0) (type default))
@@
     (stroke (width 0) (type default))
   )
-  (wire (pts (xy 46.99 100.33) (xy 46.99 121.92))
-    (stroke (width 0) (type default))
-  )
-  (wire (pts (xy 81.28 121.92) (xy 81.28 105.41))
+  (wire (pts (xy 80.01 105.41) (xy 92.71 105.41))
     (stroke (width 0) (type default))
   )
@@
     (stroke (width 0) (type default))
   )
-  (wire (pts (xy 49.53 105.41) (xy 41.91 105.41))
-    (stroke (width 0) (type default))
-  )
   (wire (pts (xy 170.18 118.11) (xy 170.18 120.65))
     (stroke (width 0) (type default))
@@
     (stroke (width 0) (type default))
   )
+  (wire (pts (xy 82.55 123.19) (xy 82.55 107.95))
+    (stroke (width 0) (type default))
+  )
   (wire (pts (xy 194.31 76.2) (xy 194.31 77.47))
     (stroke (width 0) (type default))
@@
     (stroke (width 0) (type default))
   )
+  (wire (pts (xy 44.45 105.41) (xy 44.45 123.19))
+    (stroke (width 0) (type default))
+  )
   (wire (pts (xy 181.61 72.39) (xy 184.15 72.39))
     (stroke (width 0) (type default))
   )
-  (wire (pts (xy 49.53 102.87) (xy 44.45 102.87))
-    (stroke (width 0) (type default))
-  )
   (wire (pts (xy 90.17 72.39) (xy 90.17 85.09))
     (stroke (width 0) (type default))
@@
     (stroke (width 0) (type default))
   )
-  (wire (pts (xy 49.53 100.33) (xy 46.99 100.33))
-    (stroke (width 0) (type default))
-  )
   (wire (pts (xy 148.59 67.31) (xy 151.13 67.31))
     (stroke (width 0) (type default))
   )
+  (wire (pts (xy 82.55 107.95) (xy 92.71 107.95))
+    (stroke (width 0) (type default))
+  )
   (wire (pts (xy 90.17 97.79) (xy 92.71 97.79))
     (stroke (width 0) (type default))
   )
+  (wire (pts (xy 46.99 120.65) (xy 80.01 120.65))
+    (stroke (width 0) (type default))
+  )
